File: PCB_file_measurement_card/measurement_board/kicad_v5.00/VMN/alim.kicad_sch (KiCad schematic)
At the start: 4 parts, among them J9 Screw_Terminal_01x02

Commit message: correction kicad V5.00
Parts:
- removed J9: Screw_Terminal_01x02, TerminalBlock_Phoenix:TerminalBlock_Phoenix_MKDS-1,5-2-5.08_1x02_P5.08mm_Horizontal, symbol Connector:Screw_Terminal_01x02
- renumbered Alim_5V_Digital_rasp_iso1540_mcp1 to Alim_5V_Digital_rasp_iso1540_mcp23008_current_7_click1, Alim_5V_ina282_iso1 to Alim_5V_I2C_isolator_Vmn_measurement1, Alim_analog_Vmn1 to Alim_analog_Vmn_measurement_ina128P_lm158
Connections:
- net +12V renamed 12V_Power
- net -12V renamed -12V_A
- net 12V renamed +12V_A
- net 5V renamed 5V_A
- net 5VD renamed 5V_D
- net GNDA renamed Common_A
- net GNDD renamed GND_D
- net GNDPWR renamed GND_Power
Other:
- title: (none) -> Alimentations 
