File: PCB_file_measurement_card/measurement_board/kicad_v5.00/VMN/Vmn_measurement.kicad_sch (KiCad schematic)
At the start: 21 parts, among them U2 INA128, U3 LM358, U4 1115-Adress=0X49

Commit message: last version of measurement board, with op07
Parts:
- removed D7, D8: 1N4148, Diode_THT:D_DO-35_SOD27_P7.62mm_Horizontal, symbol Diode:1N4148
- removed R9: 20 Mohms, Resistor_THT:R_Axial_DIN0204_L3.6mm_D1.6mm_P7.62mm_Horizontal, symbol Device:R
- removed U2: INA128, Package_DIP:DIP-8_W7.62mm, symbol Amplifier_Instrumentation:INA128
- removed U3: LM358, Package_DIP:DIP-8_W7.62mm, symbol Amplifier_Operational:LM358
- added C11, C13: 100nF, Capacitor_THT:C_Disc_D8.0mm_W2.5mm_P5.00mm, symbol Device:C_Small
- added C12, C14: 10uF, Capacitor_THT:CP_Radial_D6.3mm_P2.50mm, symbol Device:C_Polarized_Small
- added D7, D8: BAT86, Diode_THT:D_DO-35_SOD27_P7.62mm_Horizontal, symbol Diode:BAT86
- added RV1, RV2, RV3: R_Potentiometer, Potentiometer_THT:Potentiometer_Bourns_3296W_Vertical, symbol Device:R_Potentiometer
- added U2, U6, U7: OP07, Package_DIP:DIP-8_W7.62mm, symbol Amplifier_Operational:OP07
Connections:
- net +12V_A: now also C13.1, C14.1, D7.1 (K), RV1.2, RV2.2, RV3.2, U2.7 (V+), U6.7 (V+), U7.7 (V+)
- net -12V_A: now also C11.1, C12.2, D8.2 (A), U2.4 (V-), U6.4 (V-), U7.4 (V-)
- net Electrode_M: now also D7.2 (A), D8.1 (K), U2.3 (+)
- net at D5.2 (A), D6.1 (K), R4.2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: now also U6.6
- net at R4.1: now also U6.2 (-)
- net at R3.1: now also U2.2 (-), U2.6, U6.3 (+)
- net at R3.2, R5.1: now also U7.2 (-)
- net at D3.2 (A), D4.1 (K), R5.2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: now also U7.6
- net Electrode_N renamed GNDA
- net GNDA: now also C11.2, C12.1, C13.2, C14.2, U7.3 (+)
- new net: RV3.3, U7.1 (VOS)
- new net: RV3.1, U7.8 (VOS)
- new net: RV1.3, U2.1 (VOS)
- new net: RV1.1, U2.8 (VOS)
- new net: RV2.1, U6.8 (VOS)
- new net: RV2.3, U6.1 (VOS)
- no-connect marks 7 -> 5
Other:
- moved on the sheet: C3, C4, C5, C6, C7, C9, D3, D4, D5, D6, R4
