File: PCB_file_measurement_card/measurement_board/measurement_board_22_11/Current_injection_and_measurement.kicad_sch (KiCad schematic)
At the start: 13 parts, among them J12 Conn_01x08_Female, J14 Conn_01x02_Female, J15 Conn_01x08_Female, J20 shunt +, J21 shunt -, K3 AQY212EH, K4 AQY212EH, K5 AQY212EH, K6 AQY212EH, U5 1115-Adress=0X48

Commit message: update
Parts:
- R8: value 2 -> 2 ohms
Changed lines of the file:
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@@
       (effects (font (size 1.27 1.27)) (justify left))
     )
-    (property "Value" "2" (id 1) (at 120.65 68.5799 0)
+    (property "Value" "2 ohms" (id 1) (at 120.65 68.5799 0)
       (effects (font (size 1.27 1.27)) (justify left))
     )
