File: PCB_file_measurement_card/measurement_board/measurement_board_22_11/IHM.kicad_sch (KiCad schematic)
At the start: 8 parts

Commit message: update
Parts:
- R10, R11, R12, R13: value 330 -> 330 ohms
Changed lines of the file:
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@@
     (in_bom yes) (on_board yes) (fields_autoplaced)
     (property "Reference" "R10" (id 0) (at 129.54 58.42 90))
-    (property "Value" "330" (id 1) (at 129.54 60.96 90))
+    (property "Value" "330 ohms" (id 1) (at 129.54 60.96 90))
     (property "Footprint" "Resistor_THT:R_Axial_DIN0207_L6.3mm_D2.5mm_P7.62mm_Horizontal" (id 2) (at 129.54 66.548 90)
       (effects (font (size 1.27 1.27)) hide)
@@
     (in_bom yes) (on_board yes) (fields_autoplaced)
     (property "Reference" "R13" (id 0) (at 129.54 99.06 90))
-    (property "Value" "330" (id 1) (at 129.54 101.6 90))
+    (property "Value" "330 ohms" (id 1) (at 129.54 101.6 90))
     (property "Footprint" "Resistor_THT:R_Axial_DIN0207_L6.3mm_D2.5mm_P7.62mm_Horizontal" (id 2) (at 129.54 107.188 90)
       (effects (font (size 1.27 1.27)) hide)
@@
     (in_bom yes) (on_board yes) (fields_autoplaced)
     (property "Reference" "R12" (id 0) (at 129.54 86.36 90))
-    (property "Value" "330" (id 1) (at 129.54 88.9 90))
+    (property "Value" "330 ohms" (id 1) (at 129.54 88.9 90))
     (property "Footprint" "Resistor_THT:R_Axial_DIN0207_L6.3mm_D2.5mm_P7.62mm_Horizontal" (id 2) (at 129.54 94.488 90)
       (effects (font (size 1.27 1.27)) hide)
@@
     (in_bom yes) (on_board yes) (fields_autoplaced)
     (property "Reference" "R11" (id 0) (at 129.54 71.12 90))
-    (property "Value" "330" (id 1) (at 129.54 73.66 90))
+    (property "Value" "330 ohms" (id 1) (at 129.54 73.66 90))
     (property "Footprint" "Resistor_THT:R_Axial_DIN0207_L6.3mm_D2.5mm_P7.62mm_Horizontal" (id 2) (at 129.54 79.248 90)
       (effects (font (size 1.27 1.27)) hide)
