File: PCB_file_measurement_card/measurement_board/measurement_board_22_11/Vmn_measurement.kicad_sch (KiCad schematic)
At the start: 28 parts, among them U2 OP07, U4 1115-Adress=0X49, U6 OP07, U7 OP07

Commit message: update
Parts:
- RV1, RV2, RV3: value R_Potentiometer -> 10K
Changed lines of the file:
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@@
     (in_bom yes) (on_board yes) (fields_autoplaced)
     (property "Reference" "RV3" (id 0) (at 160.02 154.94 90))
-    (property "Value" "R_Potentiometer" (id 1) (at 160.02 157.48 90))
+    (property "Value" "10K" (id 1) (at 160.02 157.48 90))
     (property "Footprint" "Potentiometer_THT:Potentiometer_Bourns_3296W_Vertical" (id 2) (at 160.02 161.29 0)
       (effects (font (size 1.27 1.27)) hide)
@@
   )
   (symbol (lib_id "Device:R_Potentiometer") (at 157.48 66.04 270) (unit 1)
-    (in_bom yes) (on_board yes) (fields_autoplaced)
+    (in_bom yes) (on_board yes)
     (property "Reference" "RV2" (id 0) (at 157.48 59.69 90))
-    (property "Value" "R_Potentiometer" (id 1) (at 157.48 62.23 90))
+    (property "Value" "10K" (id 1) (at 157.48 62.23 90))
     (property "Footprint" "Potentiometer_THT:Potentiometer_Bourns_3296W_Vertical" (id 2) (at 157.48 66.04 0)
       (effects (font (size 1.27 1.27)) hide)
@@
     (in_bom yes) (on_board yes) (fields_autoplaced)
     (property "Reference" "RV1" (id 0) (at 102.87 111.76 90))
-    (property "Value" "R_Potentiometer" (id 1) (at 102.87 114.3 90))
+    (property "Value" "10K" (id 1) (at 102.87 114.3 90))
     (property "Footprint" "Potentiometer_THT:Potentiometer_Bourns_3296W_Vertical" (id 2) (at 102.87 118.11 0)
       (effects (font (size 1.27 1.27)) hide)
