File: PCB_file_measurement_card/measurement_board/measurement_board_22_11/alim.kicad_sch (KiCad schematic)
At the start: 3 parts

Commit message: update
Parts:
- Alim_5V_Digital_rasp_iso1540_mcp23008_current_7_click1: Arrow Price/Stock (none) -> https://www.mouser.fr/ProductDetail/TRACO-Power/THD-15-1211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
Changed lines of the file:
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@@
       (effects (font (size 1.27 1.27)) (justify left) hide)
     )
-    (property "Arrow Price/Stock" "" (id 11) (at 128.27 137.16 0)
+    (property "Arrow Price/Stock" "https://www.mouser.fr/ProductDetail/TRACO-Power/THD-15-1211N?qs=ckJk83FOD0X2IyoEoPcnmg%3D%3D" (id 11) (at 128.27 137.16 0)
       (effects (font (size 1.27 1.27)) (justify left) hide)
     )
