File: PCB_file_measurement_card/measurement_board/measurement_board_22_11/measurement_board_22_11.kicad_pcb (KiCad board)
At the start: 2 copper layers, 235 x 124 mm, 86 parts, among them J1 DSP_out_12v_GND, J10 DSP+, J11 Screw_Terminal_VMN, J12 Conn_01x08_Female, J14 Conn_01x02_Female, J15 Conn_01x08_Female, J16 RX_bat, J17 DSP GND, J18 Conn_01x01, J19 Conn_01x01, J2 DPS5005_input_0_to_50V, J20 shunt +, J21 shunt -, J3 Screw_Terminal_AB, J4 Conn_01x08_Female, J5 Conn_01x04_Female, J6 Conn_01x08_Female, J7 Raspberry_Pi_2_3, J8 Connector_I2C_for_mux_or_tools, J9 TX_bat, K1 G5LE-1, K2 G5LE-1, K3 AQY212EH, K4 AQY212EH, K5 AQY212EH, K6 AQY212EH, Q1 ZVN4206ASTZ, Q2 ZVN4206ASTZ, U1 MCP23008-xP, U2 OP07, U3 24LC02, U4 1115-Adress=0X49, U5 1115-Adress=0X48, U6 OP07, U7 OP07

Commit message: update
Parts:
- removed the R9 at (44.0, 79.2)
- J18: value Conn_01x01 -> ELEC_M
- J19: value Conn_01x01 -> ELEC_N
- R10, R11, R12, R13: value 330 -> 330 ohms
- R14, R9: value R -> 4K7; footprint Resistor_THT:R_Axial_DIN0207_L6.3mm_D2.5mm_P7.62mm_Horizontal -> Resistor_THT:R_Axial_DIN0204_L3.6mm_D1.6mm_P7.62mm_Horizontal
- R8: value 2 -> 2 ohms
- RV1, RV2, RV3: value R_Potentiometer -> 10K
- moved J12 23.0 mm to (105.0, 144.0)
- moved J15 23.0 mm to (105.0, 121.0)
- moved R9 5.64 mm to (218.4, 123.2)
- moved R14 2.47 mm to (218.4, 113.0)
Routing:
- net 5VD: track 370.1 -> 333.5 mm
- net AN: track 76.5 -> 87.6 mm
- net SCL1: track 185.8 -> 181.2 mm
- net SDA1: track 203.1 -> 205.3 mm
