File: PCB_file_measurement_card/measurement_board/measurement_board_22_11/measurement_board_22_11.kicad_sch (KiCad schematic)
At the start: 21 parts, among them J1 DSP_out_12v_GND, J10 DSP+, J11 Screw_Terminal_VMN, J16 RX_bat, J17 DSP GND, J18 Conn_01x01, J19 Conn_01x01, J2 DPS5005_input_0_to_50V, J3 Screw_Terminal_AB, J4 Conn_01x08_Female, J5 Conn_01x04_Female, J6 Conn_01x08_Female, J7 Raspberry_Pi_2_3, J8 Connector_I2C_for_mux_or_tools, J9 TX_bat, U1 MCP23008-xP, U3 24LC02

Commit message: update
Parts:
- J18: value Conn_01x01 -> ELEC_M
- J19: value Conn_01x01 -> ELEC_N
- R14: value R -> 4K7; footprint (none) -> Resistor_THT:R_Axial_DIN0204_L3.6mm_D1.6mm_P7.62mm_Horizontal
- R9: value R -> 4K7; footprint Resistor_THT:R_Axial_DIN0411_L9.9mm_D3.6mm_P12.70mm_Horizontal -> Resistor_THT:R_Axial_DIN0204_L3.6mm_D1.6mm_P7.62mm_Horizontal
- U3: footprint (none) -> Package_DIP:DIP-8_W7.62mm
Changed lines of the file:
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@@
       (effects (font (size 1.27 1.27)) (justify left))
     )
-    (property "Value" "R" (id 1) (at 274.32 64.7699 90)
-      (effects (font (size 1.27 1.27)) (justify left))
-    )
-    (property "Footprint" "" (id 2) (at 270.002 63.5 90)
+    (property "Value" "4K7" (id 1) (at 274.32 64.77 90)
+      (effects (font (size 1.27 1.27)) (justify left))
+    )
+    (property "Footprint" "Resistor_THT:R_Axial_DIN0204_L3.6mm_D1.6mm_P7.62mm_Horizontal" (id 2) (at 270.002 63.5 90)
       (effects (font (size 1.27 1.27)) hide)
     )
@@
       (effects (font (size 1.27 1.27)) (justify left))
     )
-    (property "Value" "R" (id 1) (at 265.43 64.77 90)
-      (effects (font (size 1.27 1.27)) (justify left))
-    )
-    (property "Footprint" "Resistor_THT:R_Axial_DIN0411_L9.9mm_D3.6mm_P12.70mm_Horizontal" (id 2) (at 266.192 63.5 90)
+    (property "Value" "4K7" (id 1) (at 265.43 64.77 90)
+      (effects (font (size 1.27 1.27)) (justify left))
+    )
+    (property "Footprint" "Resistor_THT:R_Axial_DIN0204_L3.6mm_D1.6mm_P7.62mm_Horizontal" (id 2) (at 266.192 63.5 90)
       (effects (font (size 1.27 1.27)) hide)
     )
@@
       (effects (font (size 1.27 1.27)) (justify left))
     )
-    (property "Footprint" "" (id 2) (at 255.27 73.66 0)
+    (property "Footprint" "Package_DIP:DIP-8_W7.62mm" (id 2) (at 255.27 73.66 0)
       (effects (font (size 1.27 1.27)) hide)
     )
@@
       (effects (font (size 1.27 1.27)) (justify left))
     )
-    (property "Value" "Conn_01x01" (id 1) (at 152.4 167.64 0)
+    (property "Value" "ELEC_N" (id 1) (at 152.4 167.64 0)
       (effects (font (size 1.27 1.27)) (justify left))
     )
@@
     (in_bom yes) (on_board yes)
     (property "Reference" "J18" (id 0) (at 133.35 162.56 0))
-    (property "Value" "Conn_01x01" (id 1) (at 132.08 167.64 0))
+    (property "Value" "ELEC_M" (id 1) (at 132.08 167.64 0))
     (property "Footprint" "Connector_PinHeader_2.54mm:PinHeader_1x01_P2.54mm_Vertical" (id 2) (at 133.35 165.1 0)
       (effects (font (size 1.27 1.27)) hide)
@@
     )
     (path "/e43d9875-30d8-42be-b597-937041f64229"
-      (reference "J18") (unit 1) (value "Conn_01x01") (footprint "Connector_PinHeader_2.54mm:PinHeader_1x01_P2.54mm_Vertical")
+      (reference "J18") (unit 1) (value "ELEC_M") (footprint "Connector_PinHeader_2.54mm:PinHeader_1x01_P2.54mm_Vertical")
     )
     (path "/b0244d42-b96a-453a-8071-d44b0d002616"
-      (reference "J19") (unit 1) (value "Conn_01x01") (footprint "Connector_PinHeader_2.54mm:PinHeader_1x01_P2.54mm_Vertical")
+      (reference "J19") (unit 1) (value "ELEC_N") (footprint "Connector_PinHeader_2.54mm:PinHeader_1x01_P2.54mm_Vertical")
     )
     (path "/3a1d549c-401c-4ddf-9a51-4b7588f9097f/84230fd6-e150-4f3f-bd4d-d1c8399a3759"
@@
     )
     (path "/3a1d549c-401c-4ddf-9a51-4b7588f9097f/fbe7548e-b89f-429b-9c09-7d2f7071b3e6"
-      (reference "R8") (unit 1) (value "2") (footprint "Resistor_THT:R_Axial_DIN0414_L11.9mm_D4.5mm_P20.32mm_Horizontal")
+      (reference "R8") (unit 1) (value "2 ohms") (footprint "Resistor_THT:R_Axial_DIN0414_L11.9mm_D4.5mm_P20.32mm_Horizontal")
     )
     (path "/9512a014-4352-43ff-a923-aca975320903"
-      (reference "R9") (unit 1) (value "R") (footprint "Resistor_THT:R_Axial_DIN0411_L9.9mm_D3.6mm_P12.70mm_Horizontal")
+      (reference "R9") (unit 1) (value "4K7") (footprint "Resistor_THT:R_Axial_DIN0204_L3.6mm_D1.6mm_P7.62mm_Horizontal")
     )
     (path "/b5055e4e-7413-40b3-89ed-dfdcecf2a97c/391691a6-fcd4-4ca7-9873-979363fe3f9a"
-      (reference "R10") (unit 1) (value "330") (footprint "Resistor_THT:R_Axial_DIN0207_L6.3mm_D2.5mm_P7.62mm_Horizontal")
+      (reference "R10") (unit 1) (value "330 ohms") (footprint "Resistor_THT:R_Axial_DIN0207_L6.3mm_D2.5mm_P7.62mm_Horizontal")
     )
     (path "/b5055e4e-7413-40b3-89ed-dfdcecf2a97c/dfa32e0f-9711-4e45-bfaa-7b800931e99e"
-      (reference "R11") (unit 1) (value "330") (footprint "Resistor_THT:R_Axial_DIN0207_L6.3mm_D2.5mm_P7.62mm_Horizontal")
+      (reference "R11") (unit 1) (value "330 ohms") (footprint "Resistor_THT:R_Axial_DIN0207_L6.3mm_D2.5mm_P7.62mm_Horizontal")
     )
     (path "/b5055e4e-7413-40b3-89ed-dfdcecf2a97c/c38c6d6c-fdb8-443a-aff0-ec2d5a0c19a0"
-      (reference "R12") (unit 1) (value "330") (footprint "Resistor_THT:R_Axial_DIN0207_L6.3mm_D2.5mm_P7.62mm_Horizontal")
+      (reference "R12") (unit 1) (value "330 ohms") (footprint "Resistor_THT:R_Axial_DIN0207_L6.3mm_D2.5mm_P7.62mm_Horizontal")
     )
     (path "/b5055e4e-7413-40b3-89ed-dfdcecf2a97c/957ddafd-3bca-4184-a9f5-92364c1f0df3"
-      (reference "R13") (unit 1) (value "330") (footprint "Resistor_THT:R_Axial_DIN0207_L6.3mm_D2.5mm_P7.62mm_Horizontal")
+      (reference "R13") (unit 1) (value "330 ohms") (footprint "Resistor_THT:R_Axial_DIN0207_L6.3mm_D2.5mm_P7.62mm_Horizontal")
     )
     (path "/319a0bf8-8f59-4e9f-8ad6-bad733c8c759"
-      (reference "R14") (unit 1) (value "R") (footprint "Resistor_THT:R_Axial_DIN0411_L9.9mm_D3.6mm_P12.70mm_Horizontal")
+      (reference "R14") (unit 1) (value "4K7") (footprint "Resistor_THT:R_Axial_DIN0204_L3.6mm_D1.6mm_P7.62mm_Horizontal")
     )
     (path "/b2026999-6d31-4d17-9f3d-996babd42897/eddcd997-356c-4d0a-b454-1e807ee28ce4"
-      (reference "RV1") (unit 1) (value "R_Potentiometer") (footprint "Potentiometer_THT:Potentiometer_Bourns_3296W_Vertical")
+      (reference "RV1") (unit 1) (value "10K") (footprint "Potentiometer_THT:Potentiometer_Bourns_3296W_Vertical")
     )
     (path "/b2026999-6d31-4d17-9f3d-996babd42897/6d56deda-84e0-4cff-9869-b9c8085f0e5a"
-      (reference "RV2") (unit 1) (value "R_Potentiometer") (footprint "Potentiometer_THT:Potentiometer_Bourns_3296W_Vertical")
+      (reference "RV2") (unit 1) (value "10K") (footprint "Potentiometer_THT:Potentiometer_Bourns_3296W_Vertical")
     )
     (path "/b2026999-6d31-4d17-9f3d-996babd42897/590bae90-4282-4179-a48b-0815bc090c3b"
-      (reference "RV3") (unit 1) (value "R_Potentiometer") (footprint "Potentiometer_THT:Potentiometer_Bourns_3296W_Vertical")
+      (reference "RV3") (unit 1) (value "10K") (footprint "Potentiometer_THT:Potentiometer_Bourns_3296W_Vertical")
     )
     (path "/9692e08d-7b1f-4dfb-891d-67e2a7a88347"
