File: PCB_file_measurement_card/measurement_board/mb.2024.0.0/Relay_switch_dsp.kicad_sch (KiCad schematic)
At the start: 8 parts, among them K1 G5LE-1, K2 G5LE-1, Q1 ZVN4206ASTZ, Q2 ZVN4206ASTZ

Commit message: rename file with the tag version
Parts:
- Q1, Q2: footprint Package_TO_SOT_THT:TO-92L_Inline -> Package_TO_SOT_THT:TO-92L_Wide
Changed lines of the file:
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@@
       (effects (font (size 1.27 1.27)) (justify left))
     )
-    (property "Footprint" "Package_TO_SOT_THT:TO-92L_Inline" (id 2) (at 102.87 132.08 0)
+    (property "Footprint" "Package_TO_SOT_THT:TO-92L_Wide" (id 2) (at 102.87 132.08 0)
       (effects (font (size 1.27 1.27)) (justify left) hide)
     )
@@
       (effects (font (size 1.27 1.27)) (justify left))
     )
-    (property "Footprint" "Package_TO_SOT_THT:TO-92L_Inline" (id 2) (at 102.87 83.82 0)
+    (property "Footprint" "Package_TO_SOT_THT:TO-92L_Wide" (id 2) (at 102.87 83.82 0)
       (effects (font (size 1.27 1.27)) (justify left) hide)
     )

Commit message: update
Connections:
- net GNDD: now also Q1.1, Q2.1, R1.1; no longer Q1.3, Q2.3, R1.2
- net MCP_GP2: now also R1.2; no longer R1.1
- net at D2.2 (A), K2.2: now also Q2.3; no longer Q2.1
- net at D1.2 (A), K1.2: now also Q1.3; no longer Q1.1
Other:
- moved on the sheet: R1, R2
Changed lines of the file:
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@@
     (title "Relay_switch_dsp")
   )
+  (junction (at 115.57 120.65) (diameter 0) (color 0 0 0 0)
+  )
   (junction (at 115.57 57.15) (diameter 0) (color 0 0 0 0)
   )
-  (junction (at 99.06 90.17) (diameter 0) (color 0 0 0 0)
-  )
-  (junction (at 87.63 130.81) (diameter 0) (color 0 0 0 0)
-  )
   (junction (at 115.57 105.41) (diameter 0) (color 0 0 0 0)
   )
-  (junction (at 87.63 82.55) (diameter 0) (color 0 0 0 0)
-  )
-  (junction (at 99.06 138.43) (diameter 0) (color 0 0 0 0)
-  )
-  (junction (at 115.57 120.65) (diameter 0) (color 0 0 0 0)
+  (junction (at 83.82 82.55) (diameter 0) (color 0 0 0 0)
   )
   (junction (at 115.57 72.39) (diameter 0) (color 0 0 0 0)
+  )
+  (junction (at 86.36 130.81) (diameter 0) (color 0 0 0 0)
   )
   (no_connect (at 140.97 57.15))
@@
     (stroke (width 0) (type default) (color 0 0 0 0))
   )
-  (wire (pts (xy 99.06 135.89) (xy 99.06 138.43))
-    (stroke (width 0) (type default) (color 0 0 0 0))
-  )
-  (wire (pts (xy 99.06 90.17) (xy 99.06 93.98))
+  (wire (pts (xy 83.82 72.39) (xy 99.06 72.39))
     (stroke (width 0) (type default) (color 0 0 0 0))
   )
@@
     (stroke (width 0) (type default) (color 0 0 0 0))
   )
-  (wire (pts (xy 99.06 120.65) (xy 115.57 120.65))
-    (stroke (width 0) (type default) (color 0 0 0 0))
-  )
-  (wire (pts (xy 87.63 82.55) (xy 91.44 82.55))
+  (wire (pts (xy 99.06 87.63) (xy 115.57 87.63))
     (stroke (width 0) (type default) (color 0 0 0 0))
   )
@@
     (stroke (width 0) (type default) (color 0 0 0 0))
   )
-  (wire (pts (xy 99.06 87.63) (xy 99.06 90.17))
+  (wire (pts (xy 115.57 135.89) (xy 115.57 120.65))
+    (stroke (width 0) (type default) (color 0 0 0 0))
+  )
+  (wire (pts (xy 86.36 123.19) (xy 86.36 120.65))
+    (stroke (width 0) (type default) (color 0 0 0 0))
+  )
+  (wire (pts (xy 115.57 87.63) (xy 115.57 72.39))
     (stroke (width 0) (type default) (color 0 0 0 0))
   )
@@
     (stroke (width 0) (type default) (color 0 0 0 0))
   )
-  (wire (pts (xy 87.63 130.81) (xy 91.44 130.81))
-    (stroke (width 0) (type default) (color 0 0 0 0))
-  )
-  (wire (pts (xy 99.06 72.39) (xy 115.57 72.39))
-    (stroke (width 0) (type default) (color 0 0 0 0))
-  )
-  (wire (pts (xy 99.06 138.43) (xy 99.06 142.24))
+  (wire (pts (xy 63.5 130.81) (xy 86.36 130.81))
+    (stroke (width 0) (type default) (color 0 0 0 0))
+  )
+  (wire (pts (xy 83.82 82.55) (xy 91.44 82.55))
     (stroke (width 0) (type default) (color 0 0 0 0))
   )
@@
     (stroke (width 0) (type default) (color 0 0 0 0))
   )
+  (wire (pts (xy 63.5 82.55) (xy 83.82 82.55))
+    (stroke (width 0) (type default) (color 0 0 0 0))
+  )
   (wire (pts (xy 115.57 50.8) (xy 115.57 57.15))
     (stroke (width 0) (type default) (color 0 0 0 0))
@@
     (stroke (width 0) (type default) (color 0 0 0 0))
   )
-  (wire (pts (xy 63.5 82.55) (xy 87.63 82.55))
+  (wire (pts (xy 99.06 135.89) (xy 115.57 135.89))
     (stroke (width 0) (type default) (color 0 0 0 0))
   )
@@
     (stroke (width 0) (type default) (color 0 0 0 0))
   )
+  (wire (pts (xy 86.36 120.65) (xy 99.06 120.65))
+    (stroke (width 0) (type default) (color 0 0 0 0))
+  )
   (wire (pts (xy 115.57 68.58) (xy 115.57 72.39))
     (stroke (width 0) (type default) (color 0 0 0 0))
   )
-  (wire (pts (xy 99.06 90.17) (xy 87.63 90.17))
+  (wire (pts (xy 86.36 130.81) (xy 91.44 130.81))
     (stroke (width 0) (type default) (color 0 0 0 0))
   )
@@
     (stroke (width 0) (type default) (color 0 0 0 0))
   )
+  (wire (pts (xy 83.82 74.93) (xy 83.82 72.39))
+    (stroke (width 0) (type default) (color 0 0 0 0))
+  )
   (wire (pts (xy 115.57 72.39) (xy 133.35 72.39))
     (stroke (width 0) (type default) (color 0 0 0 0))
   )
-  (wire (pts (xy 99.06 138.43) (xy 87.63 138.43))
-    (stroke (width 0) (type default) (color 0 0 0 0))
-  )
   (wire (pts (xy 115.57 116.84) (xy 115.57 120.65))
     (stroke (width 0) (type default) (color 0 0 0 0))
   )
-  (wire (pts (xy 63.5 130.81) (xy 87.63 130.81))
-    (stroke (width 0) (type default) (color 0 0 0 0))
-  )
   (hierarchical_label "out_GND_DSP" (shape output) (at 146.05 50.8 0)
     (effects (font (size 1.27 1.27)) (justify left))
@@
     (effects (font (size 1.27 1.27)) (justify left))
   )
-  (hierarchical_label "GNDD" (shape input) (at 99.06 142.24 0)
+  (hierarchical_label "GNDD" (shape input) (at 99.06 120.65 90)
     (effects (font (size 1.27 1.27)) (justify left))
   )
@@
     (effects (font (size 1.27 1.27)) (justify right))
   )
-  (hierarchical_label "GNDD" (shape input) (at 99.06 93.98 0)
+  (hierarchical_label "GNDD" (shape input) (at 99.06 72.39 90)
     (effects (font (size 1.27 1.27)) (justify left))
   )
@@
     (pin "2")
   )
-  (symbol (lib_id "Device:R") (at 87.63 86.36 0) (unit 1)
+  (symbol (lib_id "Device:R") (at 83.82 78.74 0) (unit 1)
     (in_bom yes) (on_board yes)
-    (property "Reference" "R1" (id 0) (at 85.09 85.09 90)
-      (effects (font (size 1.27 1.27)) (justify left))
-    )
-    (property "Value" "100k" (id 1) (at 87.63 87.63 90)
-      (effects (font (size 1.27 1.27)) (justify left))
-    )
-    (property "Footprint" "Resistor_THT:R_Axial_DIN0207_L6.3mm_D2.5mm_P7.62mm_Horizontal" (id 2) (at 85.852 86.36 90)
-      (effects (font (size 1.27 1.27)) hide)
-    )
-    (property "Datasheet" "~" (id 3) (at 87.63 86.36 0)
-      (effects (font (size 1.27 1.27)) hide)
-    )
-    (pin "1")
-    (pin "2")
-  )
-  (symbol (lib_id "Device:R") (at 87.63 134.62 0) (unit 1)
+    (property "Reference" "R1" (id 0) (at 81.28 77.47 90)
+      (effects (font (size 1.27 1.27)) (justify left))
+    )
+    (property "Value" "100k" (id 1) (at 83.82 71.12 90)
+      (effects (font (size 1.27 1.27)) (justify left))
+    )
+    (property "Footprint" "Resistor_THT:R_Axial_DIN0207_L6.3mm_D2.5mm_P7.62mm_Horizontal" (id 2) (at 82.042 78.74 90)
+      (effects (font (size 1.27 1.27)) hide)
+    )
+    (property "Datasheet" "~" (id 3) (at 83.82 78.74 0)
+      (effects (font (size 1.27 1.27)) hide)
+    )
+    (pin "1")
+    (pin "2")
+  )
+  (symbol (lib_id "Device:R") (at 86.36 127 180) (unit 1)
     (in_bom yes) (on_board yes)
-    (property "Reference" "R2" (id 0) (at 85.09 133.35 90)
-      (effects (font (size 1.27 1.27)) (justify left))
-    )
-    (property "Value" "100k" (id 1) (at 87.63 135.89 90)
-      (effects (font (size 1.27 1.27)) (justify left))
-    )
-    (property "Footprint" "Resistor_THT:R_Axial_DIN0207_L6.3mm_D2.5mm_P7.62mm_Horizontal" (id 2) (at 85.852 134.62 90)
-      (effects (font (size 1.27 1.27)) hide)
-    )
-    (property "Datasheet" "~" (id 3) (at 87.63 134.62 0)
-      (effects (font (size 1.27 1.27)) hide)
-    )
+    (property "Reference" "R2" (id 0) (at 88.9 128.27 90)
+      (effects (font (size 1.27 1.27)) (justify left))
+    )
+    (property "Value" "100k" (id 1) (at 86.36 125.73 90)
+      (effects (font (size 1.27 1.27)) (justify left))
+    )
+    (property "Footprint" "Resistor_THT:R_Axial_DIN0207_L6.3mm_D2.5mm_P7.62mm_Horizontal" (id 2) (at 88.138 127 90)
+      (effects (font (size 1.27 1.27)) hide)
+    )
+    (property "Datasheet" "~" (id 3) (at 86.36 127 0)
+      (effects (font (size 1.27 1.27)) hide)
+    )
