File: mb.2024.0.0/mb.2024.0.0.kicad_pcb (KiCad board)
At the start: 2 copper layers, 247.8 x 124 mm, 95 parts, among them J1 DSP_out_12v_GND, J10 DSP+, J11 Screw_Terminal_VMN, J12 Conn_01x08_Female, J14 Conn_01x02_Female, J15 Conn_01x08_Female, J16 RX_bat, J17 DSP GND, J18 ELEC_M, J19 ELEC_N, J2 DPS5005_input_0_to_50V, J20 shunt +, J21 shunt -, J3 Screw_Terminal_AB, J4 Conn_01x08_Female, J5 Conn_01x04_Female, J6 Conn_01x08_Female, J7 Raspberry_Pi_2_3, J8 Connector_I2C_for_mux_or_tools, J9 TX_bat, K1 G5LE-1, K2 G5LE-1, K3 G5LE-1, K4 G5LE-1, K5 G5LE-1, K6 G5LE-1, Q1 ZVN4206ASTZ, Q2 ZVN4206ASTZ, Q3 ZVN4206ASTZ, Q4 ZVN4206ASTZ, Q5 ZVN4206ASTZ, Q6 ZVN4206ASTZ, U1 MCP23008-xP, U2 OP07, U3 24LC02, U4 1115-Adress=0X49, U5 1115-Adress=0X48, U6 OP07, U7 OP07

Commit message: update
Parts:
- added J13: Connector_I2C_for_mux, Connector_IDC:IDC-Header_2x03_P2.54mm_Vertical, F.Cu at (250.9, 81.3)
- J8: value Connector_I2C_for_mux_or_tools -> Connector_I2C_for_MCP23008
Connections:
- J7 pad 15: unconnected-(J7-Pad15) -> SDA3
- J7 pad 16: unconnected-(J7-Pad16) -> SCL3
Routing:
- net SDA3: track 0.00 -> 41.4 mm
- net SCL3: track 0.00 -> 33.2 mm
- net 5VD: track 472.7 -> 504.3 mm
- net Net-(D10-Pad2): track 22.2 -> 23.4 mm
