File: mb.2024.0.0/mb.2024.0.0.kicad_sch (KiCad schematic)
At the start: 21 parts, among them J1 DSP_out_12v_GND, J10 DSP+, J11 Screw_Terminal_VMN, J16 RX_bat, J17 DSP GND, J18 ELEC_M, J19 ELEC_N, J2 DPS5005_input_0_to_50V, J3 Screw_Terminal_AB, J4 Conn_01x08_Female, J5 Conn_01x04_Female, J6 Conn_01x08_Female, J7 Raspberry_Pi_2_3, J8 Connector_I2C_for_mux_or_tools, J9 TX_bat, U1 MCP23008-xP, U3 24LC02

Commit message: update
Parts:
- added J13: Connector_I2C_for_mux, Connector_IDC:IDC-Header_2x03_P2.54mm_Vertical, symbol Connector_Generic:Conn_02x03_Top_Bottom
- J8: value Connector_I2C_for_mux_or_tools -> Connector_I2C_for_MCP23008
Connections:
- net 5VD: now also J13.6 (Pin_6)
- net GNDD: now also J13.5 (Pin_5)
- net SDA3: now reaches J7.15 (GPIO22)
- net SDA3: now also J13.3 (Pin_3)
- net SCL3: now reaches J7.16 (GPIO23)
- net SCL3: now also J13.1 (Pin_1)
Changed lines of the file:
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@@
   (no_connect (at 246.38 50.8))
   (no_connect (at 246.38 43.18))
+  (no_connect (at 182.88 77.47))
+  (no_connect (at 195.58 74.93))
   (no_connect (at 220.98 88.9))
   (no_connect (at 208.28 91.44))
@@
   (no_connect (at 200.66 25.4))
   (no_connect (at 203.2 25.4))
-  (no_connect (at 205.74 25.4))
-  (no_connect (at 208.28 25.4))
   (no_connect (at 213.36 25.4))
   (no_connect (at 215.9 25.4))
@@
     (stroke (width 0) (type default) (color 0 0 0 0))
   )
+  (wire (pts (xy 208.28 24.13) (xy 208.28 25.4))
+    (stroke (width 0) (type default) (color 0 0 0 0))
+  )
   (wire (pts (xy 33.02 55.88) (xy 33.02 52.07))
     (stroke (width 0) (type default) (color 0 0 0 0))
@@
     (stroke (width 0) (type default) (color 0 0 0 0))
   )
+  (wire (pts (xy 205.74 24.13) (xy 205.74 25.4))
+    (stroke (width 0) (type default) (color 0 0 0 0))
+  )
   (wire (pts (xy 125.73 91.44) (xy 137.16 91.44))
     (stroke (width 0) (type default) (color 0 0 0 0))
@@
     (stroke (width 0) (type default) (color 0 0 0 0))
   )
+  (wire (pts (xy 195.58 77.47) (xy 205.74 77.47))
+    (stroke (width 0) (type default) (color 0 0 0 0))
+  )
   (wire (pts (xy 232.41 153.67) (xy 232.41 148.59))
     (stroke (width 0) (type default) (color 0 0 0 0))
@@
     )
   )
+  (global_label "SDA3" (shape bidirectional) (at 208.28 24.13 90) (fields_autoplaced)
+    (effects (font (size 1.27 1.27)) (justify left))
+    (property "Intersheet References" "${INTERSHEET_REFS}" (id 0) (at 208.2006 16.9393 90)
+      (effects (font (size 1.27 1.27)) (justify left) hide)
+    )
+  )
   (global_label "5VA" (shape input) (at 210.82 110.49 90) (fields_autoplaced)
     (effects (font (size 1.27 1.27)) (justify left))
@@
     )
   )
+  (global_label "SDA3" (shape bidirectional) (at 182.88 80.01 180) (fields_autoplaced)
+    (effects (font (size 1.27 1.27)) (justify right))
+    (property "Intersheet References" "${INTERSHEET_REFS}" (id 0) (at 175.6893 80.0894 0)
+      (effects (font (size 1.27 1.27)) (justify right) hide)
+    )
+  )
+  (global_label "SCL3" (shape bidirectional) (at 205.74 24.13 90) (fields_autoplaced)
+    (effects (font (size 1.27 1.27)) (justify left))
+    (property "Intersheet References" "${INTERSHEET_REFS}" (id 0) (at 205.6606 16.9998 90)
+      (effects (font (size 1.27 1.27)) (justify left) hide)
+    )
+  )
   (global_label "5VA" (shape input) (at 154.94 138.43 0) (fields_autoplaced)
     (effects (font (size 1.27 1.27)) (justify left))
@@
     )
   )
+  (global_label "5VD" (shape input) (at 195.58 80.01 0) (fields_autoplaced)
+    (effects (font (size 1.27 1.27)) (justify left))
+    (property "Intersheet References" "${INTERSHEET_REFS}" (id 0) (at 201.5612 79.9306 0)
+      (effects (font (size 1.27 1.27)) (justify left) hide)
+    )
+  )
   (global_label "-12V_A" (shape input) (at 88.9 138.43 180) (fields_autoplaced)
     (effects (font (size 1.27 1.27)) (justify right))
@@
     (effects (font (size 1.27 1.27)) (justify right))
     (property "Intersheet References" "${INTERSHEET_REFS}" (id 0) (at 15.8507 83.7406 0)
+      (effects (font (size 1.27 1.27)) (justify right) hide)
+    )
+  )
+  (global_label "SCL3" (shape bidirectional) (at 182.88 74.93 180) (fields_autoplaced)
+    (effects (font (size 1.27 1.27)) (justify right))
+    (property "Intersheet References" "${INTERSHEET_REFS}" (id 0) (at 175.7498 75.0094 0)
       (effects (font (size 1.27 1.27)) (justify right) hide)
     )
@@
     (in_bom yes) (on_board yes) (fields_autoplaced)
     (property "Reference" "J8" (id 0) (at 214.63 82.55 0))
-    (property "Value" "Connector_I2C_for_mux_or_tools" (id 1) (at 214.63 85.09 0))
+    (property "Value" "Connector_I2C_for_MCP23008" (id 1) (at 214.63 85.09 0))
     (property "Footprint" "Connector_IDC:IDC-Header_2x03_P2.54mm_Vertical" (id 2) (at 213.36 91.44 0)
       (effects (font (size 1.27 1.27)) hide)
@@
     )
     (property "Datasheet" "" (id 3) (at 161.29 157.48 0)
+      (effects (font (size 1.27 1.27)) hide)
+    )
+    (pin "1")
+  )
+  (symbol (lib_id "power:GNDD") (at 205.74 77.47 0) (unit 1)
+    (in_bom yes) (on_board yes) (fields_autoplaced)
+    (property "Reference" "#PWR0109" (id 0) (at 205.74 83.82 0)
+      (effects (font (size 1.27 1.27)) hide)
+    )
+    (property "Value" "GNDD" (id 1) (at 205.74 82.55 0))
+    (property "Footprint" "" (id 2) (at 205.74 77.47 0)
+      (effects (font (size 1.27 1.27)) hide)
+    )
+    (property "Datasheet" "" (id 3) (at 205.74 77.47 0)
       (effects (font (size 1.27 1.27)) hide)
     )
@@
     (pin "1")
   )
+  (symbol (lib_id "Connector_Generic:Conn_02x03_Top_Bottom") (at 187.96 77.47 0) (unit 1)
+    (in_bom yes) (on_board yes) (fields_autoplaced)
+    (property "Reference" "J13" (id 0) (at 189.23 68.58 0))
+    (property "Value" "Connector_I2C_for_mux" (id 1) (at 189.23 71.12 0))
+    (property "Footprint" "Connector_IDC:IDC-Header_2x03_P2.54mm_Vertical" (id 2) (at 187.96 77.47 0)
+      (effects (font (size 1.27 1.27)) hide)
+    )
+    (property "Datasheet" "~" (id 3) (at 187.96 77.47 0)
+      (effects (font (size 1.27 1.27)) hide)
+    )
+    (pin "1")
+    (pin "2")
+    (pin "3")
+    (pin "4")
+    (pin "5")
+    (pin "6")
+  )
   (sheet (at 21.59 153.67) (size 43.18 24.13) (fields_autoplaced)
     (stroke (width 0.1524) (type solid) (color 0 0 0 0))
@@
       (reference "#PWR0108") (unit 1) (value "GNDD") (footprint "")
     )
+    (path "/6dfea346-b001-4920-aeaf-dae095291621"
+      (reference "#PWR0109") (unit 1) (value "GNDD") (footprint "")
+    )
     (path "/9f60bb1d-ca92-41d5-b592-f34396aa7479/e59d3cfa-2d20-458f-8209-a7dc300d5c82"
       (reference "Alim_5V_Digital_rasp_iso1540_mcp23008_current_7_click1") (unit 1) (value "THD_15-1211N") (footprint "THD_15-1211N:THD151211N")
@@
     )
     (path "/49058ded-2ed2-473c-ba90-e52b2c428f78"
-      (reference "J8") (unit 1) (value "Connector_I2C_for_mux_or_tools") (footprint "Connector_IDC:IDC-Header_2x03_P2.54mm_Vertical")
+      (reference "J8") (unit 1) (value "Connector_I2C_for_MCP23008") (footprint "Connector_IDC:IDC-Header_2x03_P2.54mm_Vertical")
     )
     (path "/69f7acd3-c534-45d5-925d-06ac5b005f91"
@@
       (reference "J12") (unit 1) (value "Conn_01x08_Female") (footprint "Connector_PinHeader_2.54mm:PinHeader_1x08_P2.54mm_Vertical")
     )
+    (path "/fa8c8cec-67e2-4fe6-a7c0-01f39434a05f"
+      (reference "J13") (unit 1) (value "Connector_I2C_for_mux") (footprint "Connector_IDC:IDC-Header_2x03_P2.54mm_Vertical")
+    )
     (path "/3a1d549c-401c-4ddf-9a51-4b7588f9097f/8dd326d7-fec8-441e-97a0-1ac0d41eba6c"
