File: PCB_boards/mux_boards/mux.2024.0.1/mux.2024.0.1.kicad_pcb (KiCad board)
At the start: 2 copper layers, 140 x 350 mm, 199 parts, among them K1 G5LE-1-VD, K10 G5LE-1-VD, K11 G5LE-1-VD, K12 G5LE-1-VD, K13 G5LE-1-VD, K14 G5LE-1-VD, K15 G5LE-1-VD, K16 G5LE-1-VD, K17 G5LE-1-VD, K18 G5LE-1-VD, K19 G5LE-1-VD, K2 G5LE-1-VD, K20 G5LE-1-VD, K21 G5LE-1-VD, K22 G5LE-1-VD, K23 G5LE-1-VD, K24 G5LE-1-VD, K25 G5LE-1-VD, K26 G5LE-1-VD, K27 G5LE-1-VD, K28 G5LE-1-VD, K29 G5LE-1-VD, K3 G5LE-1-VD, K30 G5LE-1-VD, K31 G5LE-1-VD, K32 G5LE-1-VD, K4 G5LE-1-VD, K5 G5LE-1-VD, K6 G5LE-1-VD, K7 G5LE-1-VD, K8 G5LE-1-VD, K9 G5LE-1-VD, Q1 STP16NF06L, Q10 STP16NF06L, Q11 STP16NF06L, Q12 STP16NF06L, Q13 STP16NF06L, Q14 STP16NF06L, Q15 STP16NF06L, Q16 STP16NF06L, Q17 STP16NF06L, Q18 STP16NF06L, Q19 STP16NF06L, Q2 STP16NF06L, Q20 STP16NF06L, Q21 STP16NF06L, Q22 STP16NF06L, Q23 STP16NF06L, Q24 STP16NF06L, Q25 STP16NF06L, Q26 STP16NF06L, Q27 STP16NF06L, Q28 STP16NF06L, Q29 STP16NF06L, Q3 STP16NF06L, Q30 STP16NF06L, Q31 STP16NF06L, Q32 STP16NF06L, Q4 STP16NF06L, Q5 STP16NF06L, Q6 STP16NF06L, Q7 STP16NF06L, Q8 STP16NF06L, Q9 STP16NF06L, U1 MCP23017_SP, U2 MCP23017_SP

Commit message: Updates MUX.2024.0.1 design
Routing:
- net Role xx: track 259.0 -> 344.4 mm
- net Role yy: track 315.2 -> 379.9 mm
- net Net-(D31-Pad2): track 23.7 -> 32.0 mm
Changed lines of the file:
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@@
   (segment (start 145.038992 187.5) (end 145.038992 179.337227) (width 0.5) (layer "B.Cu") (net 55))
   (segment (start 145.038992 142.373007) (end 141.098991 138.433006) (width 0.5) (layer "B.Cu") (net 56))
+  (segment (start 141.098991 138.433006) (end 145.73796 138.433006) (width 0.5) (layer "B.Cu") (net 56))
   (segment (start 132.18024 138.433006) (end 131.420241 137.673007) (width 0.5) (layer "B.Cu") (net 56))
   (segment (start 145.038992 150.5) (end 145.038992 142.373007) (width 0.5) (layer "B.Cu") (net 56))
   (segment (start 141.098991 138.433006) (end 132.18024 138.433006) (width 0.5) (layer "B.Cu") (net 56))
+  (segment (start 145.73796 138.433006) (end 148.333992 141.029038) (width 0.5) (layer "B.Cu") (net 56))
   (segment (start 132.153574 101.468786) (end 131.420241 100.735453) (width 0.5) (layer "B.Cu") (net 57))
   (segment (start 145.038992 113.8) (end 145.038992 105.408787) (width 0.5) (layer "B.Cu") (net 57))
@@
   (segment (start 112.773892 92.5) (end 145.970241 59.303651) (width 2) (layer "B.Cu") (net 59))
   (segment (start 73.051491 106.701666) (end 80.733575 106.701666) (width 2) (layer "B.Cu") (net 59))
+  (segment (start 134.110241 87.616676) (end 133.460241 88.266676) (width 2) (layer "F.Cu") (net 60))
   (segment (start 131.387951 337.010288) (end 136.069752 341.692089) (width 2) (layer "F.Cu") (net 60))
+  (segment (start 135 112.5) (end 135 123.664471) (width 2) (layer "F.Cu") (net 60))
   (segment (start 128.735241 335.422752) (end 130.322777 337.010288) (width 2) (layer "F.Cu") (net 60))
   (segment (start 128.735241 143.28026) (end 128.735241 158.7) (width 2) (layer "F.Cu") (net 60))
+  (segment (start 133.460241 88.266676) (end 134.110241 88.916676) (width 2) (layer "F.Cu") (net 60))
+  (segment (start 130.5 109.5) (end 132 109.5) (width 2) (layer "F.Cu") (net 60))
   (segment (start 128.735241 306.7) (end 128.735241 335.422752) (width 2) (layer "F.Cu") (net 60))
   (segment (start 130.322777 337.010288) (end 131.387951 337.010288) (width 2) (layer "F.Cu") (net 60))
+  (segment (start 150.990241 60.95) (end 149.970241 61.97) (width 2) (layer "F.Cu") (net 60))
   (segment (start 133.460241 162.141784) (end 132.177025 162.141784) (width 2) (layer "F.Cu") (net 60))
+  (segment (start 131.414547 103.385453) (end 129.9 104.9) (width 2) (layer "F.Cu") (net 60))
   (segment (start 131.514579 199.079338) (end 128.735241 196.3) (width 2) (layer "F.Cu") (net 60))
+  (segment (start 134.110241 88.916676) (end 134.110241 101.793119) (width 2) (layer "F.Cu") (net 60))
   (segment (start 133.460241 125.20423) (end 134.109752 125.853741) (width 2) (layer "F.Cu") (net 60))
   (segment (start 136.069752 341.692089) (end 136.069752 344.220044) (width 2) (layer "F.Cu") (net 60))
+  (segment (start 132.517907 103.385453) (end 131.414547 103.385453) (width 2) (layer "F.Cu") (net 60))
   (segment (start 133.460242 309.892) (end 131.927241 309.892) (width 2) (layer "F.Cu") (net 60))
   (segment (start 133.460241 236.016892) (end 131.052133 236.016892) (width 2) (layer "F.Cu") (net 60))
   (segment (start 136.069752 344.220044) (end 133.460242 346.829554) (width 2) (layer "F.Cu") (net 60))
   (segment (start 134.109752 138.825489) (end 131.911745 141.023496) (width 2) (layer "F.Cu") (net 60))
+  (segment (start 135 123.664471) (end 133.460241 125.20423) (width 2) (layer "F.Cu") (net 60))
+  (segment (start 149.970241 63.770001) (end 134.110241 79.630001) (width 2) (layer "F.Cu") (net 60))
+  (segment (start 150.990241 53.3) (end 150.990241 60.95) (width 2) (layer "F.Cu") (net 60))
   (segment (start 128.735241 270.3) (end 128.735241 306.7) (width 2) (layer "F.Cu") (net 60))
   (segment (start 132.177025 162.141784) (end 128.735241 158.7) (width 2) (layer "F.Cu") (net 60))
+  (segment (start 129.9 104.9) (end 129.9 108.9) (width 2) (layer "F.Cu") (net 60))
   (segment (start 130.992005 141.023496) (end 128.735241 143.28026) (width 2) (layer "F.Cu") (net 60))
   (segment (start 134.109752 125.853741) (end 134.109752 138.825489) (width 2) (layer "F.Cu") (net 60))
+  (segment (start 134.110241 101.793119) (end 132.517907 103.385453) (width 2) (layer "F.Cu") (net 60))
   (segment (start 131.052133 236.016892) (end 128.735241 233.7) (width 2) (layer "F.Cu") (net 60))
+  (segment (start 132 109.5) (end 135 112.5) (width 2) (layer "F.Cu") (net 60))
+  (segment (start 149.970241 61.97) (end 149.970241 63.770001) (width 2) (layer "F.Cu") (net 60))
   (segment (start 131.389687 272.954446) (end 128.735241 270.3) (width 2) (layer "F.Cu") (net 60))
   (segment (start 128.735241 196.3) (end 128.735241 233.7) (width 2) (layer "F.Cu") (net 60))
@@
   (segment (start 128.735241 158.7) (end 128.735241 196.3) (width 2) (layer "F.Cu") (net 60))
   (segment (start 131.911745 141.023496) (end 130.992005 141.023496) (width 2) (layer "F.Cu") (net 60))
+  (segment (start 134.110241 79.630001) (end 134.110241 87.616676) (width 2) (layer "F.Cu") (net 60))
+  (segment (start 129.9 108.9) (end 130.5 109.5) (width 2) (layer "F.Cu") (net 60))
   (segment (start 133.460241 199.079338) (end 131.514579 199.079338) (width 2) (layer "F.Cu") (net 60))
   (segment (start 131.927241 309.892) (end 128.735241 306.7) (width 2) (layer "F.Cu") (net 60))
@@
   (segment (start 135.362234 143.673007) (end 137.835241 141.2) (width 2) (layer "F.Cu") (net 61))
   (segment (start 133.420241 143.673007) (end 135.362234 143.673007) (width 2) (layer "F.Cu") (net 61))
+  (segment (start 133.420241 106.735453) (end 136.510241 103.645453) (width 2) (layer "F.Cu") (net 61))
   (segment (start 138.469263 323.965978) (end 138.469263 287.034022) (width 2) (layer "F.Cu") (net 61))
   (segment (start 138.469263 287.034022) (end 138.469263 250.034022) (width 2) (layer "F.Cu") (net 61))
@@
   (segment (start 156.070241 53.3) (end 156.070241 51.12) (width 2) (layer "F.Cu") (net 61))
   (segment (start 133.420241 328.360777) (end 134.074464 328.360777) (width 2) (layer "F.Cu") (net 61))
+  (segment (start 136.510241 103.645453) (end 136.510241 80.624113) (width 2) (layer "F.Cu") (net 61))
   (segment (start 133.420241 180.015) (end 138.469263 174.965978) (width 2) (layer "F.Cu") (net 61))
+  (segment (start 156.070241 61.064113) (end 156.070241 53.3) (width 2) (layer "F.Cu") (net 61))
+  (segment (start 136.670241 106.735453) (end 133.420241 106.735453) (width 2) (layer "F.Cu") (net 61))
   (segment (start 138.469263 174.965978) (end 138.469263 141.834022) (width 2) (layer "F.Cu") (net 61))
   (segment (start 138.469263 360.249312) (end 138.469263 323.965978) (width 2) (layer "F.Cu") (net 61))
   (segment (start 133.520241 217.548115) (end 133.95517 217.548115) (width 2) (layer "F.Cu") (net 61))
   (segment (start 133.420241 180.610561) (end 133.420241 180.015) (width 2) (layer "F.Cu") (net 61))
+  (segment (start 136.510241 80.624113) (end 156.070241 61.064113) (width 2) (layer "F.Cu") (net 61))
   (segment (start 134.017616 254.485669) (end 138.469263 250.034022) (width 2) (layer "F.Cu") (net 61))
   (segment (start 133.420241 291.423223) (end 134.080062 291.423223) (width 2) (layer "F.Cu") (net 61))
   (segment (start 133.95517 217.548115) (end 138.469263 213.034022) (width 2) (layer "F.Cu") (net 61))
+  (segment (start 137.835241 107.900453) (end 136.670241 106.735453) (width 2) (layer "F.Cu") (net 61))
+  (segment (start 137.835241 141.2) (end 137.835241 107.900453) (width 2) (layer "F.Cu") (net 61))
   (segment (start 138.469263 141.834022) (end 137.835241 141.2) (width 2) (layer "F.Cu") (net 61))
-  (segment (start 137.835241 141.2) (end 137.835241 111.150453) (width 2) (layer "F.Cu") (net 61))
-  (segment (start 137.835241 111.150453) (end 133.420241 106.735453) (width 2) (layer "F.Cu") (net 61))
   (segment (start 57.126925 382.947066) (end 62.758991 377.315) (width 0.5) (layer "F.Cu") (net 62))
   (segment (start 39 91.795241) (end 39 380) (width 0.5) (layer "F.Cu") (net 62))
