File: PCB_boards/measurement_boards/mb.2024.0.2/Vmn_measurement.kicad_sch (KiCad schematic)
At the start: 39 parts, among them J27 Screw_Terminal_01x03, U10 DG411xJ, U2 OP07, U4 1085, U6 OP07, U7 REF03GP, U8 MCP23008-xP, U9 OP07

Commit message: update measurement board
Parts:
- removed C5: 10uF, Capacitor_THT:CP_Radial_D6.3mm_P2.50mm, symbol Device:C_Polarized_Small
- removed J27: Screw_Terminal_01x03, TerminalBlock:TerminalBlock_bornier-3_P5.08mm, symbol Connector:Screw_Terminal_01x03
- added C3, C9: 10uF, Capacitor_THT:CP_Radial_D6.3mm_P2.50mm, symbol Device:C_Polarized_Small
- added C5: 100nF, Capacitor_THT:C_Disc_D8.0mm_W2.5mm_P5.00mm, symbol Device:C_Small
- added R21, R22: 4.7K, Resistor_THT:R_Axial_DIN0207_L6.3mm_D2.5mm_P7.62mm_Horizontal, symbol Device:R
Connections:
- net +12V_A: now also C3.1, C5.1, C9.1
- net 5VA: now also R21.2, R22.2
- net GNDA: now also C3.2, C5.2, C9.2
- net SCL2: now also R21.1
- net SDA2: now also R22.1
- no-connect marks 9 -> 12
Other:
- note added: "2.5V de référence"
- note added: "Ampli suiveur"
- note added: "Gain unitaire ou Gain = 0.5"
- note added: "Isolation de la masse"
- note added: "additionneur pour offset de 2.5V"
- note removed: "2.5V offset adder"
- note removed: "2.5V reference"
- note removed: "Follower amp"
- note removed: "Ground insulation"
- note removed: "Unit gain or Gain = 0.5"
- moved on the sheet: R5

Commit message: correction DPS, add dischage resistor, remove 63 warning on the schemtic, remove 7 errors in schematics change resistor designation, update pcb
Parts:
- removed C3, C9: 10uF, Capacitor_THT:CP_Radial_D6.3mm_P2.50mm, symbol Device:C_Polarized_Small
- removed C5: 100nF, Capacitor_THT:C_Disc_D8.0mm_W2.5mm_P5.00mm, symbol Device:C_Small
- removed R21, R22: 4.7K, Resistor_THT:R_Axial_DIN0207_L6.3mm_D2.5mm_P7.62mm_Horizontal, symbol Device:R
- added C5: 10uF, Capacitor_THT:CP_Radial_D6.3mm_P2.50mm, symbol Device:C_Polarized_Small
- added J27: Screw_Terminal_01x03, TerminalBlock:TerminalBlock_bornier-3_P5.08mm, symbol Connector:Screw_Terminal_01x03
Connections:
- net +12V_A: now also C5.1
- net GNDA: now also C5.2
- net at U4.1 (A3): now also J27.1 (Pin_1)
- net at U4.2 (A2): now also J27.2 (Pin_2)
- net at U4.3 (A1): now also J27.3 (Pin_3)
- no-connect marks 12 -> 9
Other:
- note added: "2.5V offset adder"
- note added: "2.5V reference"
- note added: "Follower amp"
- note added: "Ground insulation"
- note added: "Unit gain or Gain = 0.5"
- note removed: "2.5V de référence"
- note removed: "Ampli suiveur"
- note removed: "Gain unitaire ou Gain = 0.5"
- note removed: "Isolation de la masse"
- note removed: "additionneur pour offset de 2.5V"
- moved on the sheet: R5
