File: PCB_boards/measurement_boards/mb.2024.0.2/Current_injection_and_measurement.kicad_sch (KiCad schematic)
At the start: 28 parts, among them J12 Conn_01x08_Socket, J14 Conn_01x02_Socket, J15 Conn_01x08_Socket, J20 shunt +, J21 shunt -, K3 G5LE-1, K4 G5LE-1, K5 G5LE-1, K6 G5LE-1, K7 G5LE-1, Q3 ZVN4206ASTZ, Q4 ZVN4206ASTZ, Q5 ZVN4206ASTZ, Q6 ZVN4206ASTZ, Q7 ZVN4206ASTZ, U5 1085

Commit message: update measurement board
Connections:
- net Input_DPS_+_alim: now also K7.3; no longer K7.4
Changed lines of the file:
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@@
   )
   (no_connect (at 133.35 171.45))
-  (no_connect (at 266.7 25.4))
+  (no_connect (at 261.62 25.4))
   (no_connect (at 161.29 161.29))
   (no_connect (at 252.73 132.08))
@@
     (stroke (width 0) (type default))
   )
-  (wire (pts (xy 280.67 19.05) (xy 261.62 19.05))
+  (wire (pts (xy 280.67 19.05) (xy 266.7 19.05))
     (stroke (width 0) (type default))
   )
@@
     (stroke (width 0) (type default))
   )
-  (wire (pts (xy 261.62 19.05) (xy 261.62 25.4))
-    (stroke (width 0) (type default))
-  )
   (wire (pts (xy 229.87 66.04) (xy 229.87 72.39))
     (stroke (width 0) (type default))
@@
     (stroke (width 0) (type default))
   )
+  (wire (pts (xy 266.7 19.05) (xy 266.7 25.4))
+    (stroke (width 0) (type default))
+  )
