File: PCB_boards/mux_boards/mux.2024.0.2/mux.2024.0.2.kicad_pcb (KiCad board)
At the start: 2 copper layers, 140 x 350 mm, 199 parts, among them K1 G5LE-1-VD, K10 G5LE-1-VD, K11 G5LE-1-VD, K12 G5LE-1-VD, K13 G5LE-1-VD, K14 G5LE-1-VD, K15 G5LE-1-VD, K16 G5LE-1-VD, K17 G5LE-1-VD, K18 G5LE-1-VD, K19 G5LE-1-VD, K2 G5LE-1-VD, K20 G5LE-1-VD, K21 G5LE-1-VD, K22 G5LE-1-VD, K23 G5LE-1-VD, K24 G5LE-1-VD, K25 G5LE-1-VD, K26 G5LE-1-VD, K27 G5LE-1-VD, K28 G5LE-1-VD, K29 G5LE-1-VD, K3 G5LE-1-VD, K30 G5LE-1-VD, K31 G5LE-1-VD, K32 G5LE-1-VD, K4 G5LE-1-VD, K5 G5LE-1-VD, K6 G5LE-1-VD, K7 G5LE-1-VD, K8 G5LE-1-VD, K9 G5LE-1-VD, Q1 STP16NF06L, Q10 STP16NF06L, Q11 STP16NF06L, Q12 STP16NF06L, Q13 STP16NF06L, Q14 STP16NF06L, Q15 STP16NF06L, Q16 STP16NF06L, Q17 STP16NF06L, Q18 STP16NF06L, Q19 STP16NF06L, Q2 STP16NF06L, Q20 STP16NF06L, Q21 STP16NF06L, Q22 STP16NF06L, Q23 STP16NF06L, Q24 STP16NF06L, Q25 STP16NF06L, Q26 STP16NF06L, Q27 STP16NF06L, Q28 STP16NF06L, Q29 STP16NF06L, Q3 STP16NF06L, Q30 STP16NF06L, Q31 STP16NF06L, Q32 STP16NF06L, Q4 STP16NF06L, Q5 STP16NF06L, Q6 STP16NF06L, Q7 STP16NF06L, Q8 STP16NF06L, Q9 STP16NF06L, U1 MCP23017_SP, U2 MCP23017_SP

Commit message: Fix mux2024 pcb missing R10-gate ZVN connection
Routing:
- net E10x: track 94.2 -> 100.5 mm
- removed copper zone on F.Cu, net GND

Commit message: Updates zone on MUX_2024.0.2 pcb
Routing:
- added copper zone on F.Cu, net GND
Changed lines of the file:
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@@
 		(net 18)
 		(net_name "GND")
-		(layer "B.Cu")
+		(layers "F&B.Cu")
 		(hatch edge 0.5)
 		(connect_pads
